Commit message: added camera_depth frame

File: launch/panda_camera.urdf.xacro (robot description, xacro)
@@ -6,10 +6,30 @@
                       joint_limits="${xacro.load_yaml('$(find franka_description)/robots/panda/joint_limits.yaml')}">
   </xacro:franka_robot>
-  <!-- camera_link -->
-  <link name="camera_link"/>
+  <!-- camera_joint -->
   <joint name="camera_joint" type="fixed">
     <origin xyz="0.05 0 0" rpy="-${pi} -${pi/2.0} 0"/>
     <parent link="panda_hand"/>
     <child link="camera_link"/>
+  </joint>
+  <!-- camera_link -->
+  <link name="camera_link">
+    <visual>
+        <origin xyz="0 0 0" rpy="-${pi} -${pi/2.0} 0"/>
+        <geometry>
+            <box size="0.05 0.05 0.05"/>
+        </geometry>
+    </visual>
+    <inertial>
+        <mass value="0.0001" />
+        <origin xyz="0 0 0" rpy="0 0 0"/>
+        <inertia ixx="0.0000001" ixy="0" ixz="0" iyy="0.0000001" iyz="0" izz="0.0000001" />
+    </inertial>
+  </link>
+  <!-- camera_depth_link -->
+  <link name="camera_depth_link" />
+  <joint name="camera_depth_module" type="fixed">
+    <origin xyz="0 0 0" rpy="-1.57 0 -1.57" />
+    <parent link="camera_link" />
+    <child  link="camera_depth_link" />
   </joint>
   <gazebo reference="camera_link"> <!-- your_camera_link -->
@@ -18,9 +38,10 @@
       <visualize>true</visualize>
       <camera>
+          <pose>0 0 0 0 0 0</pose>
           <horizontal_fov>1.047</horizontal_fov>
           <image>
               <width>640</width>
               <height>480</height>
-              <format>R8G8B8</format>
+              <format>B8G8R8</format>
           </image>
           <depth_camera>
@@ -34,7 +55,7 @@
           <baseline>0.2</baseline>
           <alwaysOn>true</alwaysOn>
-              <updateRate>0.0</updateRate>
-              <cameraName>camera</cameraName>
-              <frameName>camera_link</frameName>
+          <updateRate>0.0</updateRate>
+          <cameraName>camera</cameraName>
+          <frameName>camera_depth_link</frameName>
           <imageTopicName>rgb/image_raw</imageTopicName>
           <depthImageTopicName>depth/image_raw</depthImageTopicName>
@@ -43,10 +64,10 @@
           <depthImageCameraInfoTopicName>depth/camera_info</depthImageCameraInfoTopicName>
           <pointCloudCutoff>0.4</pointCloudCutoff>
-              <hackBaseline>0.07</hackBaseline>
-              <distortionK1>0.0</distortionK1>
-              <distortionK2>0.0</distortionK2>
-              <distortionK3>0.0</distortionK3>
-              <distortionT1>0.0</distortionT1>
-              <distortionT2>0.0</distortionT2>
+          <hackBaseline>0.07</hackBaseline>
+          <distortionK1>0.0</distortionK1>
+          <distortionK2>0.0</distortionK2>
+          <distortionK3>0.0</distortionK3>
+          <distortionT1>0.0</distortionT1>
+          <distortionT2>0.0</distortionT2>
           <CxPrime>0.0</CxPrime>
           <Cx>0.0</Cx>
