Commit message: panda urdf update

File: launch/urdf/panda_camera.urdf.xacro (robot description, xacro)
@@ -2,12 +2,34 @@
 <robot xmlns:xacro="http://www.ros.org/wiki/xacro" name="panda">
   <xacro:include filename="$(find franka_description)/robots/common/franka_robot.xacro"/>
+  <!-- Name for this robot -->
   <xacro:arg name="arm_id" default="panda" />
+  <!-- Should a franka_gripper be mounted at the flange?" -->
+  <xacro:arg name="hand" default="false" />
+  <!-- Positional offset between $(arm_id)_hand -> $(arm_id)_hand_tcp [m]. Only used when hand:=true -->
+  <xacro:arg name="tcp_xyz" default="0 0 0.1034" />
+  <!-- Rotational offset between $(arm_id)_hand -> $(arm_id)_hand_tcp [rad]. Only used when hand:=true -->
+  <xacro:arg name="tcp_rpy" default="0 0 0" />
+  <!-- Is the robot being simulated in gazebo?" -->
+  <xacro:arg name="gazebo" default="false" />
+  <!-- If `gazebo` arg is set, to which frame shall $(arm_id)_link0 be parented. Empty string for not fixing at all -->
+  <xacro:arg name="parent" default="world" />
+  <!-- If `gazebo` arg is set and `parent` not empty, what position offset between `parent` & $(arm_id)_link0 -->
+  <xacro:arg name="xyz" default="0 0 0" />
+  <!-- If `gazebo` arg is set and `parent` not empty, what rotation offset between `parent` & $(arm_id)_link0 -->
+  <xacro:arg name="rpy" default="0 0 0" />
   <xacro:franka_robot arm_id="$(arg arm_id)"
-                      joint_limits="${xacro.load_yaml('$(find franka_description)/robots/panda/joint_limits.yaml')}">
+                      joint_limits="${xacro.load_yaml('$(find franka_description)/robots/panda/joint_limits.yaml')}"
+                      hand="$(arg hand)"
+                      tcp_xyz="$(arg tcp_xyz)"
+                      tcp_rpy="$(arg tcp_rpy)"
+                      gazebo="$(arg gazebo)"
+                      parent="$(arg parent)"
+                      xyz="$(arg xyz)"
+                      rpy="$(arg rpy)">
   </xacro:franka_robot>
   <!-- camera_joint -->
   <joint name="camera_joint" type="fixed">
-    <origin xyz="0.05 0 0" rpy="-${pi} -${pi/2.0} 0"/>
-    <parent link="panda_hand"/>
+    <origin xyz="0.045 -0.045 0" rpy="-${pi} -${pi/2.0} ${pi/4.0}"/>
+    <parent link="$(arg arm_id)_link7"/>
     <child link="camera_link"/>
   </joint>
@@ -17,5 +39,5 @@
         <origin xyz="0 0 0" rpy="-${pi} -${pi/2.0} 0"/>
         <geometry>
-            <box size="0.05 0.05 0.05"/>
+            <box size="0.06 0.04 0.025"/>
         </geometry>
     </visual>
@@ -77,20 +99,3 @@
     </sensor>
   </gazebo>
-  <gazebo>
-   <plugin name="gazebo_grasp_fix" filename="libgazebo_grasp_fix.so">
-        <arm>
-           <arm_name>panda</arm_name>
-           <palm_link> panda_link7  </palm_link>
-           <gripper_link> panda_leftfinger </gripper_link>
-           <gripper_link> panda_rightfinger </gripper_link>
-        </arm>
-       <forces_angle_tolerance>100</forces_angle_tolerance>
-       <update_rate>4</update_rate>
-       <grip_count_threshold>4</grip_count_threshold>
-       <max_grip_count>8</max_grip_count>
-       <release_tolerance>0.005</release_tolerance>
-       <disable_collisions_on_attach>false</disable_collisions_on_attach>
-       <contact_topic>__default_topic__</contact_topic>
-    </plugin>
-</gazebo>
 </robot>
