Commit message: updates ur5e; send_joints test

File: launch/urdf/ur5e_2f85.xacro (robot description, xacro)
@@ -9,14 +9,25 @@
     <origin xyz="0.0 0.0 0.0" rpy="0.0 0.0 0.0" />
   </joint>
-  <!-- camera_link -->
-  <link name="camera_link"/>
   <joint name="camera_joint" type="fixed">
     <!-- default toolframe: X+ left, Y+ up, Z+ front -->
-    <origin xyz="0 -0.05 0" rpy="${pi/2.0} -${pi/2.0} 0"/>
+    <origin xyz="0 -0.055 0" rpy="${pi/2.0} -${pi/2.0} 0"/>
     <parent link="tool0"/>
     <child link="camera_link"/>
   </joint>
+  <!-- camera_link -->
+  <link name="camera_link">
+    <visual>
+        <geometry>
+            <box size="0.01 0.04 0.03"/>
+        </geometry>
+    </visual>
+    <inertial>
+        <mass value="0.0001" />
+        <origin xyz="0 0 0" rpy="0 0 0"/>
+        <inertia ixx="0.0000001" ixy="0" ixz="0" iyy="0.0000001" iyz="0" izz="0.0000001" />
+    </inertial>
+  </link>
   <gazebo reference="camera_link"> <!-- your_camera_link -->
-    <sensor type="depth" name="camera1">
+    <sensor type="depth" name="camera">
       <always_on>true</always_on>
       <visualize>true</visualize>
@@ -39,5 +50,5 @@
           <alwaysOn>true</alwaysOn>
               <updateRate>10.0</updateRate>
-              <cameraName>camera1</cameraName>
+              <cameraName>camera</cameraName>
               <frameName>camera_link</frameName>
           <imageTopicName>rgb/image_raw</imageTopicName>

Commit message: depth_camera_link

File: launch/urdf/ur5e_2f85.xacro (robot description, xacro)
@@ -28,4 +28,11 @@
     </inertial>
   </link>
+  <!-- camera_depth_link -->
+  <link name="camera_depth_link" />
+  <joint name="camera_depth_module" type="fixed">
+    <origin xyz="0 0 0" rpy="-1.57 0 -1.57" />
+    <parent link="camera_link" />
+    <child  link="camera_depth_link" />
+  </joint>
   <gazebo reference="camera_link"> <!-- your_camera_link -->
     <sensor type="depth" name="camera">
@@ -37,5 +44,5 @@
               <width>640</width>
               <height>480</height>
-              <format>R8G8B8</format>
+              <format>B8G8R8</format>
           </image>
           <depth_camera>
@@ -51,5 +58,5 @@
               <updateRate>10.0</updateRate>
               <cameraName>camera</cameraName>
-              <frameName>camera_link</frameName>
+              <frameName>camera_depth_link</frameName>
           <imageTopicName>rgb/image_raw</imageTopicName>
           <depthImageTopicName>depth/image_raw</depthImageTopicName>
